File: computer.kicad_pcb (KiCad board)
At the start: 2 copper layers, 182.2 x 157.5 mm, 27 parts, among them J1 Jack-DC, J2 Conn_02x09_Counter_Clockwise, J3 Conn_02x08_Counter_Clockwise, SW1 SW_Push, U1 AS6C6264, U10 Z80CPU, U11 CD74HCT138E, U12 CD74HCT138E, U13 Z80_PIO, U14 Z80_PIO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

Commit message: update
Parts:
- removed J2: Conn_02x09_Counter_Clockwise, Connector_PinSocket_1.27mm:PinSocket_2x09_P1.27mm_Vertical
- removed U15: Z80_PIO, Package_DIP:DIP-40_W15.24mm_Socket_LongPads
- added C10: 100nF, Capacitor_THT:C_Disc_D5.0mm_W2.5mm_P2.50mm, F.Cu at (208.5, 141.0)
- added C11: 100nF, Capacitor_THT:C_Disc_D5.0mm_W2.5mm_P2.50mm, F.Cu at (233.5, 102.0)
- added C12: 100nF, Capacitor_THT:C_Disc_D5.0mm_W2.5mm_P2.50mm, F.Cu at (181.8, 61.8)
- added C13: 100nF, Capacitor_THT:C_Disc_D5.0mm_W2.5mm_P2.50mm, F.Cu at (116.5, 153.0)
- added C14: 100nF, Capacitor_THT:C_Disc_D5.0mm_W2.5mm_P2.50mm, F.Cu at (109.0, 141.0)
- added C15: 100nF, Capacitor_THT:C_Disc_D5.0mm_W2.5mm_P2.50mm, F.Cu at (259.0, 102.0)
- added C16: 100nF, Capacitor_THT:C_Disc_D5.0mm_W2.5mm_P2.50mm, F.Cu at (146.5, 153.0)
- added C17: 100nF, Capacitor_THT:C_Disc_D5.0mm_W2.5mm_P2.50mm, F.Cu at (131.0, 116.5)
- added C18: 100nF, Capacitor_THT:C_Disc_D5.0mm_W2.5mm_P2.50mm, F.Cu at (94.5, 64.5)
- added C3: 100nF, Capacitor_THT:C_Disc_D5.0mm_W2.5mm_P2.50mm, F.Cu at (258.5, 61.8)
- added C4: 100nF, Capacitor_THT:C_Disc_D5.0mm_W2.5mm_P2.50mm, F.Cu at (182.5, 102.0)
- added C5: 100nF, Capacitor_THT:C_Disc_D5.0mm_W2.5mm_P2.50mm, F.Cu at (233.0, 61.8)
- added C6: 100nF, Capacitor_THT:C_Disc_D5.0mm_W2.5mm_P2.50mm, F.Cu at (120.0, 77.0)
- added C7: 100nF, Capacitor_THT:C_Disc_D5.0mm_W2.5mm_P2.50mm, F.Cu at (208.0, 102.0)
- added C8: 100nF, Capacitor_THT:C_Disc_D5.0mm_W2.5mm_P2.50mm, F.Cu at (207.5, 61.8)
- added C9: 100nF, Capacitor_THT:C_Disc_D5.0mm_W2.5mm_P2.50mm, F.Cu at (155.0, 63.5)
- J3: footprint Connector_PinSocket_1.27mm:PinSocket_2x08_P1.27mm_Vertical -> Connector_PinSocket_2.00mm:PinSocket_2x08_P2.00mm_Vertical
- U17: footprint Connector_PinSocket_1.00mm:PinSocket_1x16_P1.00mm_Vertical -> Connector_PinSocket_2.00mm:PinSocket_1x16_P2.00mm_Vertical
- moved U14 39.0 mm to (161.0, 134.5)
- moved U16 39.0 mm to (131.2, 156.5)
- moved U18 39.0 mm to (160.2, 156.5)
- moved J3 28.0 mm to (128.5, 171.0)
- moved U12 24.3 mm to (113.8, 112.0)
- moved U17 12.9 mm to (215.0, 157.5)
Routing:
- net /CLK: track 10.2 -> 126.6 mm
- net /CPU_INT: track 0.00 -> 90.5 mm
- net /D1: track 156.6 -> 236.3 mm
- net /CPU_A13: track 0.00 -> 70.7 mm, vias 0 -> 1
- net /CPU_A12: track 156.6 -> 224.3 mm, vias 0 -> 1
- net /CPU_A11: track 156.6 -> 219.1 mm, vias 0 -> 1
- net Net-(U14-Pad15): track 0.00 -> 49.1 mm
- net /CPU_A10: track 156.6 -> 202.6 mm, vias 0 -> 1
- net /CPU_A9: track 156.6 -> 201.0 mm, vias 0 -> 1
- net Net-(U14-Pad14): track 0.00 -> 42.8 mm
- net /CPU_A8: track 156.6 -> 198.9 mm, vias 0 -> 1
- net /CPU_A7: track 156.6 -> 196.2 mm, vias 0 -> 1
- net /CPU_A6: track 156.6 -> 194.6 mm, vias 0 -> 1
- net /CPU_A5: track 156.6 -> 192.5 mm, vias 0 -> 1
- net Net-(RV1-Pad2): track 0.00 -> 35.9 mm
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- removed copper zone on B.Cu, net VCC
Other:
- copper layers 2 -> 4
- net class Default: clearance 0.2 -> 0.1; via_dia 0.8 -> 0.4; via_drill 0.4 -> 0.2
- rule trace_clearance: 0.2 -> 0.1
- rule via_min_drill: 0.3 -> 0.15
