File: computer.sch (KiCad schematic (older format))
At the start: 13 parts, among them U1 Z80CPU

Commit message: aaa
Parts:
- removed U?: NM27C256Q150, symbol chips:NM27C256Q150
- added C3: 1u, Capacitor_Tantalum_SMD:CP_EIA-2012-15_AVX-P_Pad1.30x1.05mm_HandSolder, symbol Device:C
- added R3: 100, Resistor_SMD:R_1206_3216Metric_Pad1.42x1.75mm_HandSolder, symbol Device:R
- added R4: 1k, Resistor_SMD:R_1206_3216Metric_Pad1.42x1.75mm_HandSolder, symbol Device:R
- added RV?: 10k-20k, symbol Device:R_POT
- added SW1: SW_Push, Button_Switch_THT:SW_PUSH_6mm, symbol Switch:SW_Push
- added U2: AT28C256, Package_DIP:DIP-28_W15.24mm_Socket_LongPads, symbol chips2:AT28C256
- added U4, U?: AS6C6264, Package_DIP:DIP-28_W15.24mm_Socket_LongPads, symbol chips2:AS6C6264
- added U7: Z80_PIO, Package_DIP:DIP-40_W15.24mm_Socket_LongPads, symbol computer-rescue:Z80_PIO-chips
- added U?: NHD-0420H1Z, Display:NHD-0420H1Z, symbol Display_Character:NHD-0420H1Z
- added U?: 74AUC2G04, symbol 74xGxx:74AUC2G04
- added U? (x2): 74LS15, symbol 74xx:74LS15
- C1, C2: renamed from C?; footprint (none) -> Capacitor_Tantalum_SMD:CP_EIA-2012-15_AVX-P_Pad1.30x1.05mm_HandSolder
- R1, R2: renamed from R?; footprint (none) -> Resistor_SMD:R_1206_3216Metric_Pad1.42x1.75mm_HandSolder
- U1: renamed from U?; footprint (none) -> Package_DIP:DIP-14_W7.62mm_Socket_LongPads
- U3: renamed from U1; footprint (none) -> Package_DIP:DIP-40_W15.24mm_Socket_LongPads
- U5, U6: renamed from U?; footprint (none) -> Package_DIP:DIP-40_W15.24mm_Socket_LongPads; symbol chips:Z80_PIO -> computer-rescue:Z80_PIO-chips
- Y1: renamed from Y?; footprint (none) -> Crystal:Crystal_HC52-8mm_Horizontal_1EP_style2
Connections:
- net labels added: CPU_MREQ, CPU_WR, LCD_DB0, LCD_DB1, LCD_DB2, LCD_DB3, LCD_DB4, LCD_DB5, LCD_DB6, LCD_DB7, LCD_E, LCD_RS, LCD_RW, RESET
- wire segments 41 -> 54
Other:
- note added: "EEPROM\n32,768 * 8bit words\n262,144 total bits"
- note added: "LCD 1"
- note added: "MEMORY MAP:\n===========\n\n0x0000 -> 0x7FFF = EEPROM\n0000 0000 0000 0000b -> 0111 1111 1111 1111\n\n0x8000 -> 0x9FFF = RAM 1\n1000 0000 0000 0000b -> 1001 1111 1111 1111\n\n0xa000 -> 0xbfff = RAM 2\n1010 0000 0000 0000b -> 1011 1111 1111 1111"
- note added: "RAM\n8,192 * 8bit words\n65,536 total bits"
- moved on the sheet: C1, C2, R1, R2, U3

Commit message: aaaaaaaa
Parts:
- removed U?: AS6C6264, Package_DIP:DIP-28_W15.24mm_Socket_LongPads, symbol chips2:AS6C6264
- removed U?: 74AUC2G04, symbol 74xGxx:74AUC2G04
- removed U? (x2): 74LS15, symbol 74xx:74LS15
- added D1: LED, symbol components:LED
- added J?: DB15_Female_MountingHoles, symbol Connector:DB15_Female_MountingHoles
- added Q1: 2N7000, Package_TO_SOT_THT:TO-92_Inline, symbol Transistor_FET:2N7000
- added R10, R11, R12, R5, R7, R8, R9, R? (x8): R, symbol Device:R
- added R6: 330, symbol Device:R
- added SW2, SW3, SW4, SW5, SW6, SW7, SW8, SW? (x8): SW_Push, symbol Switch:SW_Push
- U2: symbol chips2:AT28C256 -> computer-rescue:AT28C256-chips2
- U4: symbol chips2:AS6C6264 -> computer-rescue:AS6C6264-chips2
- Y1: value 4MHz -> 16MHz
- gave numbers to parts that had none: 2
Connections:
- net labels added: CLK, DSUB1, DSUB2, DSUB3, DSUB4, DSUB5, DSUB6, DSUB7, DSUB8, DSUB_1, DSUB_10, DSUB_11, DSUB_12, DSUB_13, DSUB_14, DSUB_15, DSUB_2, DSUB_3, DSUB_4, DSUB_5, DSUB_6, DSUB_7, DSUB_8, DSUB_9
- wire segments 54 -> 131
Other:
- note added: "MEMORY MAP:\n===========\n\n0x0000 -> 0x7FFF = EEPROM\n0000 0000 0000 0000b -> 0111 1111 1111 1111\n\n0x8000 -> 0x9FFF = RAM 1\n1000 0000 0000 0000b -> 1001 1111 1111 1111"
- note removed: "MEMORY MAP:\n===========\n\n0x0000 -> 0x7FFF = EEPROM\n0000 0000 0000 0000b -> 0111 1111 1111 1111\n\n0x8000 -> 0x9FFF = RAM 1\n1000 0000 0000 0000b -> 1001 1111 1111 1111\n\n0xa000 -> 0xbfff = RAM 2\n1010 0000 0000 0000b -> 1011 1111 1111 1111"
- moved on the sheet: C1, C2, C3, R1, R2, R3, R4, RV1, SW1, U3, U5, U6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

Commit message: fin
Parts:
- removed C2: 100n, Capacitor_Tantalum_SMD:CP_EIA-2012-15_AVX-P_Pad1.30x1.05mm_HandSolder, symbol Device:C
- removed D1: LED, symbol components:LED
- removed J?: DB15_Female_MountingHoles, symbol Connector:DB15_Female_MountingHoles
- removed Q1: 2N7000, Package_TO_SOT_THT:TO-92_Inline, symbol Transistor_FET:2N7000
- removed R10, R5, R8, R? (x8): R, symbol Device:R
- removed SW? (x8): SW_Push, symbol Switch:SW_Push
- removed U1: 74LS00, Package_DIP:DIP-14_W7.62mm_Socket_LongPads, symbol 74xx:74LS00
- removed U2: AT28C256, Package_DIP:DIP-28_W15.24mm_Socket_LongPads, symbol computer-rescue:AT28C256-chips2
- removed U4: AS6C6264, Package_DIP:DIP-28_W15.24mm_Socket_LongPads, symbol computer-rescue:AS6C6264-chips2
- removed Y1: 16MHz, Crystal:Crystal_HC52-8mm_Horizontal_1EP_style2, symbol Device:Crystal
- added C3, C4: 10uF, Capacitor_THT:CP_Radial_D8.0mm_P3.50mm, symbol Device:C
- added Q1, Q2, Q3, Q4: Q_NMOS_DGS, Package_TO_SOT_THT:TO-92, symbol Device:Q_NMOS_DGS
- added R12, R13, R14, R15, R16, R17, R18, R3, R4: 1k, Resistor_THT:R_Axial_DIN0204_L3.6mm_D1.6mm_P5.08mm_Horizontal, symbol Device:R
- added SW1, SW10, SW11, SW12, SW13, SW14, SW15, SW16, SW17: SW_Push, symbol Switch:SW_Push
- added U11, U13, U14, U15: AS6C6264, symbol computer-rescue:AS6C6264-chips2
- added U3, U5, U8, U9: AT28C64B, symbol chips2:AT28C64B
- added U6: CD74HCT138E, symbol chips2:CD74HCT138E
- added U7: CA56-12EWA, symbol Display_Character:CA56-12EWA
- added X1: ACO-8MHz, symbol Oscillator:ACO-xxxMHz
- C1: value 120p -> 0.01uF; footprint Capacitor_Tantalum_SMD:CP_EIA-2012-15_AVX-P_Pad1.30x1.05mm_HandSolder -> Capacitor_THT:C_Disc_D5.0mm_W2.5mm_P2.50mm
- C2: renamed from C3; footprint Capacitor_Tantalum_SMD:CP_EIA-2012-15_AVX-P_Pad1.30x1.05mm_HandSolder -> Capacitor_THT:C_Disc_D5.0mm_W2.5mm_P2.50mm
- R1, R2: value 330 -> 1k; footprint Resistor_SMD:R_1206_3216Metric_Pad1.42x1.75mm_HandSolder -> Resistor_THT:R_Axial_DIN0204_L3.6mm_D1.6mm_P5.08mm_Horizontal
- R10: renamed from R12; value R -> 1k; footprint (none) -> Resistor_THT:R_Axial_DIN0204_L3.6mm_D1.6mm_P5.08mm_Horizontal
- R11, R7, R9: value R -> 1k; footprint (none) -> Resistor_THT:R_Axial_DIN0204_L3.6mm_D1.6mm_P5.08mm_Horizontal
- R5: renamed from R4; footprint Resistor_SMD:R_1206_3216Metric_Pad1.42x1.75mm_HandSolder -> Resistor_THT:R_Axial_DIN0204_L3.6mm_D1.6mm_P5.08mm_Horizontal
- R6: value 330 -> 1k; footprint (none) -> Resistor_THT:R_Axial_DIN0204_L3.6mm_D1.6mm_P5.08mm_Horizontal
- R8: renamed from R3; footprint Resistor_SMD:R_1206_3216Metric_Pad1.42x1.75mm_HandSolder -> Resistor_THT:R_Axial_DIN0204_L3.6mm_D1.6mm_P5.08mm_Horizontal
- RV1: footprint (none) -> Potentiometer_THT:Potentiometer_Bourns_3266W_Vertical
- SW9: renamed from SW1; footprint Button_Switch_THT:SW_PUSH_6mm -> (none)
- U1: renamed from U5; footprint Package_DIP:DIP-40_W15.24mm_Socket_LongPads -> (none)
- U10: renamed from U7; footprint Package_DIP:DIP-40_W15.24mm_Socket_LongPads -> (none)
- U12: renamed from U8; footprint Display:NHD-0420H1Z -> (none)
- U2: renamed from U3; footprint Package_DIP:DIP-40_W15.24mm_Socket_LongPads -> (none)
- U4: renamed from U6; footprint Package_DIP:DIP-40_W15.24mm_Socket_LongPads -> (none)
Connections:
- net labels removed: DSUB1, DSUB2, DSUB3, DSUB4, DSUB5, DSUB6, DSUB7, DSUB8, DSUB_1, DSUB_10, DSUB_11, DSUB_12, DSUB_13, DSUB_14, DSUB_15, DSUB_2, DSUB_3, DSUB_4, DSUB_5, DSUB_6, DSUB_7, DSUB_8, DSUB_9
- wire segments 131 -> 166
Other:
- note added: "DATA\nBUS"
- note added: "EEPROM (0x0000)\n8,192 * 8bit words\n65,536 total bits"
- note added: "EEPROM (0x2000)\n8,192 * 8bit words\n65,536 total bits"
- note added: "EEPROM (4000)\n8,192 * 8bit words\n65,536 total bits"
- note added: "EEPROM (6000)\n8,192 * 8bit words\n65,536 total bits"
- note added: "LCD 4x20"
- note added: "MEMORY MAP\n==============\n\n0b0000 0000 0000 0000 -> 0b0111 1111 1111 1111\n= 0x0000 -> 0x7fff = EEPROM\n\n0b1000 0000 0000 0000 -> 0b1111 1111 1111 1111\n= 0x8000 -> 0xffff = SRAM"
- note added: "SRAM (8000)\n8,192 * 8bit words\n65,536 total bits"
- note added: "SRAM (a000)\n8,192 * 8bit words\n65,536 total bits"
- note added: "SRAM (c000)\n8,192 * 8bit words\n65,536 total bits"
- note added: "SRAM (e000)\n8,192 * 8bit words\n65,536 total bits"
- note removed: "EEPROM\n32,768 * 8bit words\n262,144 total bits"
- note removed: "LCD 1"
- note removed: "MEMORY MAP:\n===========\n\n0x0000 -> 0x7FFF = EEPROM\n0000 0000 0000 0000b -> 0111 1111 1111 1111\n\n0x8000 -> 0x9FFF = RAM 1\n1000 0000 0000 0000b -> 1001 1111 1111 1111"
- note removed: "RAM\n8,192 * 8bit words\n65,536 total bits"
- moved on the sheet: C2, R10, R5, R8, RV1, SW9, U1, U10, U12, U2, U4

Commit message: update
Parts:
- removed C3, C4: 10uF, Capacitor_THT:CP_Radial_D8.0mm_P3.50mm, symbol Device:C
- removed Q1, Q2, Q3, Q4: Q_NMOS_DGS, Package_TO_SOT_THT:TO-92, symbol Device:Q_NMOS_DGS
- removed R1, R10, R11, R12, R13, R14, R15, R16, R17, R18, R2, R3, R4, R6, R7, R9: 1k, Resistor_THT:R_Axial_DIN0204_L3.6mm_D1.6mm_P5.08mm_Horizontal, symbol Device:R
- removed R8: 100, Resistor_THT:R_Axial_DIN0204_L3.6mm_D1.6mm_P5.08mm_Horizontal, symbol Device:R
- removed SW1, SW10, SW11, SW12, SW13, SW14, SW15, SW16, SW17, SW2, SW3, SW4, SW5, SW6, SW7, SW8: SW_Push, symbol Switch:SW_Push
- removed U1, U10, U4: Z80_PIO, symbol computer-rescue:Z80_PIO-chips
- removed U12: NHD-0420H1Z, symbol Display_Character:NHD-0420H1Z
- removed U7: CA56-12EWA, symbol Display_Character:CA56-12EWA
- added J1: Jack-DC, Connector_BarrelJack:BarrelJack_CUI_PJ-063AH_Horizontal, symbol Connector:Jack-DC
- added J2: Conn_02x09_Counter_Clockwise, Connector_PinSocket_1.27mm:PinSocket_2x09_P1.27mm_Vertical, symbol Connector_Generic:Conn_02x09_Counter_Clockwise
- added J3: Conn_02x08_Counter_Clockwise, Connector_PinSocket_1.27mm:PinSocket_2x08_P1.27mm_Vertical, symbol Connector_Generic:Conn_02x08_Counter_Clockwise
- added U12: CD74HCT138E, Package_DIP:DIP-16_W7.62mm_Socket_LongPads, symbol chips2:CD74HCT138E
- added U13, U14, U15: Z80_PIO, Package_DIP:DIP-40_W15.24mm_Socket_LongPads, symbol chips2:Z80_PIO
- added U16, U18: CD74HC238E, Package_DIP:DIP-16_W7.62mm_Socket_LongPads, symbol chips2:CD74HC238E
- added U17: NHD-0420H1Z, Connector_PinSocket_1.00mm:PinSocket_1x16_P1.00mm_Vertical, symbol Display_Character:NHD-0420H1Z
- added U9: L7805, Package_TO_SOT_THT:TO-220-3_Vertical, symbol Regulator_Linear:L7805
- SW1: renamed from SW9; footprint (none) -> Button_Switch_THT:SW_PUSH_6mm_H4.3mm
- U1: renamed from U13; footprint (none) -> Package_DIP:DIP-28_W15.24mm_Socket_LongPads
- U10: renamed from U2; footprint (none) -> Package_DIP:DIP-40_W15.24mm_Socket_LongPads
- U11: renamed from U6; footprint (none) -> Package_DIP:DIP-16_W7.62mm_Socket_LongPads
- U2: renamed from U15; footprint (none) -> Package_DIP:DIP-28_W15.24mm_Socket_LongPads
- U3: renamed from U5; footprint (none) -> Package_DIP:DIP-28_W15.24mm_Socket_LongPads
- U4: renamed from U9; footprint (none) -> Package_DIP:DIP-28_W15.24mm_Socket_LongPads
- U5: renamed from U11; footprint (none) -> Package_DIP:DIP-28_W15.24mm_Socket_LongPads
- U6: renamed from U14; footprint (none) -> Package_DIP:DIP-28_W15.24mm_Socket_LongPads
- U7: renamed from U3; footprint (none) -> Package_DIP:DIP-28_W15.24mm_Socket_LongPads
- U8: footprint (none) -> Package_DIP:DIP-28_W15.24mm_Socket_LongPads
- X1: footprint (none) -> Oscillator:Oscillator_DIP-14_LargePads
- renumbered C2 to C1, C1 to C2, R5 to R1
Connections:
- net RESET is gone; now on an unnamed net: U10.26 (~RESET~)
- net CLK: now also U13.25 (CLK), U14.25 (CLK), U15.25 (CLK)
- net CPU_A0: now also U13.6 (A/B), U14.6 (A/B), U15.6 (A/B)
- net CPU_A1: now also U13.5 (C/D), U14.5 (C/D), U15.5 (C/D)
- net CPU_A2: now also U12.1 (A0)
- net CPU_A3: now also U12.2 (A1)
- net CPU_A4: now also U12.3 (A2)
- net CPU_INT: now also U13.23 (~INT), U14.23 (~INT), U15.23 (~INT)
- net CPU_IORQ: now also U13.4 (~CE), U14.4 (~CE), U15.4 (~CE)
- net CPU_M1: now also U13.37 (~M1), U14.37 (~M1), U15.37 (~M1)
- net CPU_RD: now also U13.35 (~RD), U14.35 (~RD), U15.35 (~RD)
- net D0: now also U13.19 (D0), U14.19 (D0), U15.19 (D0)
- net D1: now also U13.20 (D1), U14.20 (D1), U15.20 (D1)
- net D2: now also U13.1 (D2), U14.1 (D2), U15.1 (D2)
- net D3: now also U13.40 (D3), U14.40 (D3), U15.40 (D3)
- net D4: now also U13.39 (D4), U14.39 (D4), U15.39 (D4)
- net D5: now also U13.38 (D5), U14.38 (D5), U15.38 (D5)
- net D6: now also U13.3 (D6), U14.3 (D6), U15.3 (D6)
- net D7: now also U13.2 (D7), U14.2 (D7), U15.2 (D7)
- net GND: now also J1.2, J2.10 (Pin_10), U12.5 (~E2), U12.8 (GND), U13.11 (GND), U14.11 (GND), U15.11 (GND), U16.4 (~E1), U16.5 (~E2), U16.8 (GND), U17.1 (VSS), U17.16 (K), U18.4 (~E1), U18.5 (~E2), U18.8 (GND), U9.2 (GND); no longer C2.1, R1.1, RV1.3, U1.26 (CE2), U1.28 (VCC), U10.11 (VCC), U11.16 (VCC), U11.6 (E3), U2.26 (CE2), U2.28 (VCC), U3.28 (VCC), U4.28 (VCC), U5.26 (CE2), U5.28 (VCC), U6.26 (CE2), U6.28 (VCC), U7.28 (VCC), U8.28 (VCC), X1.14 (Vcc)
- net at C1.1, R1.2: now also SW1.2; no longer U10.28 (~RFSH~)
- net at RV1.2: now also U17.3 (VO)
- new net: U14.15 (A0), U18.1 (A0)
- new net: U14.14 (A1), U18.2 (A1)
- new net: U14.13 (A2), U18.3 (A2)
- new net: U14.27 (B0), U16.1 (A0)
- new net: U14.28 (B1), U16.2 (A1)
- new net: U14.29 (B2), U16.3 (A2)
- new net: U12.13 (~Y1), U14.36 (~IORQ)
- new net: U12.14 (~Y2), U15.36 (~IORQ)
- new net: U12.15 (~Y0), U13.36 (~IORQ)
- new net: U13.30 (B3), U17.10 (DB3)
- new net: U13.31 (B4), U17.11 (DB4)
- new net: U13.32 (B5), U17.12 (DB5)
- new net: U13.33 (B6), U17.13 (DB6)
- new net: U13.34 (B7), U17.14 (DB7)
- new net: U13.15 (A0), U17.4 (RS)
- new net: U13.14 (A1), U17.5 (R/W)
- new net: U13.13 (A2), U17.6 (E)
- new net: U13.27 (B0), U17.7 (DB0)
- new net: U13.28 (B1), U17.8 (DB1)
- new net: U13.29 (B2), U17.9 (DB2)
- new net: J2.1 (Pin_1), U15.15 (A0)
- new net: J2.11 (Pin_11), U15.34 (B7)
- new net: J2.12 (Pin_12), U15.33 (B6)
- new net: J2.13 (Pin_13), U15.32 (B5)
- new net: J2.14 (Pin_14), U15.31 (B4)
- new net: J2.15 (Pin_15), U15.30 (B3)
- new net: J2.16 (Pin_16), U15.29 (B2)
- new net: J2.17 (Pin_17), U15.28 (B1)
- new net: J2.18 (Pin_18), U15.27 (B0)
- new net: J2.2 (Pin_2), U15.14 (A1)
- new net: J2.3 (Pin_3), U15.13 (A2)
- new net: J2.4 (Pin_4), U15.12 (A3)
- new net: J2.5 (Pin_5), U15.10 (A4)
- new net: J2.6 (Pin_6), U15.9 (A5)
- new net: J2.7 (Pin_7), U15.8 (A6)
- new net: J2.8 (Pin_8), U15.7 (A7)
- new net: J1.1, U9.1 (IN)
- new net CPU_IOREQ: U12.4 (~E1)
- new net VCC: C2.1, J2.9 (Pin_9), R1.1, RV1.3, U1.26 (CE2), U1.28 (VCC), U10.11 (VCC), U11.16 (VCC), U11.6 (E3), U12.16 (VCC), U12.6 (E3), U13.26 (+5V), U14.26 (+5V), U15.26 (+5V), U16.16 (VCC), U16.6 (E3), U17.15 (A), U17.2 (VDD), U18.16 (VCC), U18.6 (E3), U2.26 (CE2), U2.28 (VCC), U3.28 (VCC), U4.28 (VCC), U5.26 (CE2), U5.28 (VCC), U6.26 (CE2), U6.28 (VCC), U7.28 (VCC), U8.28 (VCC), U9.3 (OUT), X1.14 (Vcc)
- new net kbd_in0: J3.8 (Pin_8), U16.15 (Y0)
- new net kbd_in1: J3.7 (Pin_7), U16.13 (Y1)
- new net kbd_in2: J3.6 (Pin_6), U16.14 (Y2)
- new net kbd_in3: J3.5 (Pin_5), U16.12 (Y3)
- new net kbd_in4: J3.4 (Pin_4), U16.11 (Y4)
- new net kbd_in5: J3.3 (Pin_3), U16.10 (Y5)
- new net kbd_in6: J3.2 (Pin_2), U16.9 (Y6)
- new net kbd_in7: J3.1 (Pin_1), U16.7 (Y7)
- new net kbd_out0: J3.16 (Pin_16), U18.15 (Y0)
- new net kbd_out1: J3.15 (Pin_15), U18.13 (Y1)
- new net kbd_out2: J3.14 (Pin_14), U18.14 (Y2)
- new net kbd_out3: J3.13 (Pin_13), U18.12 (Y3)
- new net kbd_out4: J3.12 (Pin_12), U18.11 (Y4)
- new net kbd_out5: J3.11 (Pin_11), U18.10 (Y5)
- new net kbd_out6: J3.10 (Pin_10), U18.9 (Y6)
- new net kbd_out7: J3.9 (Pin_9), U18.7 (Y7)
Other:
- note added: "MEMORY MAP (Total 64K memory (ROM + RAM))\n==============\n\n0b0000 0000 0000 0000 -> 0b0111 1111 1111 1111\n= 0x0000 -> 0x7fff = EEPROM\n\n0b1000 0000 0000 0000 -> 0b1111 1111 1111 1111\n= 0x8000 -> 0xffff = SRAM\n\ni.e. A15 high = RAM, A15 low = ROM"
- note removed: "MEMORY MAP\n==============\n\n0b0000 0000 0000 0000 -> 0b0111 1111 1111 1111\n= 0x0000 -> 0x7fff = EEPROM\n\n0b1000 0000 0000 0000 -> 0b1111 1111 1111 1111\n= 0x8000 -> 0xffff = SRAM"
- moved on the sheet: C1, C2, R1, SW1, X1

Commit message: update
Parts:
- removed J2: Conn_02x09_Counter_Clockwise, Connector_PinSocket_1.27mm:PinSocket_2x09_P1.27mm_Vertical, symbol Connector_Generic:Conn_02x09_Counter_Clockwise
- removed J3: Conn_02x08_Counter_Clockwise, Connector_PinSocket_1.27mm:PinSocket_2x08_P1.27mm_Vertical, symbol Connector_Generic:Conn_02x08_Counter_Clockwise
- removed U15: Z80_PIO, Package_DIP:DIP-40_W15.24mm_Socket_LongPads, symbol chips2:Z80_PIO
- removed U16, U18: CD74HC238E, Package_DIP:DIP-16_W7.62mm_Socket_LongPads, symbol chips2:CD74HC238E
- removed X1: ACO-8MHz, Oscillator:Oscillator_DIP-14_LargePads, symbol Oscillator:ACO-xxxMHz
- added C10, C11, C12, C13, C14, C15, C16, C17, C3, C4, C5, C6, C7, C8, C9: 100nF, Capacitor_THT:C_Disc_D5.0mm_W2.5mm_P2.50mm, symbol Device:C
- added R?: 1k, symbol Device:R_Small
- added RN?: 1k, symbol Device:R_Pack08
- added SW?: SW_DIP_x08, symbol Switch:SW_DIP_x08
- added X?: OSC, Oscillator:Oscillator_DIP-14, symbol Oscillator:ACO-xxxMHz
- R1: footprint Resistor_THT:R_Axial_DIN0204_L3.6mm_D1.6mm_P5.08mm_Horizontal -> Resistor_SMD:R_1206_3216Metric_Pad1.42x1.75mm_HandSolder
Connections:
- net CLK: now also X?.8 (OUT)
- net CPU_INT: now also U13.22 (IEO), R?.2
- net GND: now also C10.1, C11.1, C12.1, C13.1, C14.1, C15.1, C16.1, C17.1, C3.1, C4.1, C5.1, C6.1, C7.1, C8.1, C9.1, SW?.10, SW?.11, SW?.12, SW?.13, SW?.14, SW?.15, SW?.16, SW?.9, X?.7 (GND)
- net VCC: now also U14.24 (IEI), C10.2, C11.2, C12.2, C13.2, C14.2, C15.2, C16.2, C17.2, C3.2, C4.2, C5.2, C6.2, C7.2, C8.2, C9.2, R?.1, RN?.10 (R7.2), RN?.11 (R6.2), RN?.12 (R5.2), RN?.13 (R4.2), RN?.14 (R3.2), RN?.15 (R2.2), RN?.16 (R1.2), RN?.9 (R8.2), X?.14 (Vcc)
- net at U14.14 (A1): now also RN?.7 (R7.1), SW?.2
- net at U14.13 (A2): now also SW?.3
- net at U13.24 (IEI): now also U14.22 (IEO)
- net at U14.10 (A4): now also RN?.4 (R4.1), SW?.5
- net at U14.12 (A3): now also RN?.5 (R5.1), SW?.4
- net at U14.7 (A7): now also RN?.1 (R1.1), SW?.8
- net at U14.8 (A6): now also RN?.2 (R2.1), SW?.7
- net at U14.9 (A5): now also RN?.3 (R3.1), SW?.6
- new net: RN?.8 (R8.1), SW?.1
Other:
- note added: "ADDR\nBUS"
- note added: "Place these caps close to the chips!"
- note added: "http://z80.info/1653.htm"
- moved on the sheet: J1, RV1, U17, U9
